File: Modulo_4Reles/Modulo_4Reles.sch (KiCad schematic (older format))
At the start: 32 parts, among them J1 Digital_Inputs, J2 Conn_01x03, J3 Conn_01x03, J4 Conn_01x03, J5 Conn_01x03, J6 Conn_01x02, K1 SANYOU_SRD_Form_C, K2 SANYOU_SRD_Form_C, K3 SANYOU_SRD_Form_C, K4 SANYOU_SRD_Form_C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

Commit message: Add files via upload
Parts:
- R1, R2, R3, R7: value 330 -> 1k
Other:
- moved on the sheet: C1, C2, J1, J6
Changed lines of the file:
@@
 P 3700 3050
 F 0 "R1" V 3600 3000 50  0000 L CNN
-F 1 "330" V 3800 3000 50  0000 L CNN
+F 1 "1k" V 3800 3000 50  0000 L CNN
 F 2 "Resistor_THT:R_Axial_DIN0207_L6.3mm_D2.5mm_P10.16mm_Horizontal" H 3700 3050 50  0001 C CNN
 F 3 "~" H 3700 3050 50  0001 C CNN
@@
 L Connector:Conn_01x06_Male J1
 U 1 1 5DABD198
-P 2300 3900
-F 0 "J1" H 2406 4278 50  0000 C CNN
-F 1 "Digital_Inputs" H 2406 4187 50  0000 C CNN
-F 2 "Connector_Molex:Molex_KK-254_AE-6410-06A_1x06_P2.54mm_Vertical" H 2300 3900 50  0001 C CNN
-F 3 "~" H 2300 3900 50  0001 C CNN
-	1    2300 3900
+P 1725 3625
+F 0 "J1" H 1831 4003 50  0000 C CNN
+F 1 "Digital_Inputs" H 1831 3912 50  0000 C CNN
+F 2 "Connector_Molex:Molex_KK-254_AE-6410-06A_1x06_P2.54mm_Vertical" H 1725 3625 50  0001 C CNN
+F 3 "~" H 1725 3625 50  0001 C CNN
+	1    1725 3625
 	1    0    0    -1
 $EndComp
@@
 P 3700 5000
 F 0 "R2" V 3600 4950 50  0000 L CNN
-F 1 "330" V 3800 4950 50  0000 L CNN
+F 1 "1k" V 3800 4950 50  0000 L CNN
 F 2 "Resistor_THT:R_Axial_DIN0207_L6.3mm_D2.5mm_P10.16mm_Horizontal" H 3700 5000 50  0001 C CNN
 F 3 "~" H 3700 5000 50  0001 C CNN
@@
 P 3700 6950
 F 0 "R3" V 3600 6900 50  0000 L CNN
-F 1 "330" V 3800 6900 50  0000 L CNN
+F 1 "1k" V 3800 6900 50  0000 L CNN
 F 2 "Resistor_THT:R_Axial_DIN0207_L6.3mm_D2.5mm_P10.16mm_Horizontal" H 3700 6950 50  0001 C CNN
 F 3 "~" H 3700 6950 50  0001 C CNN
@@
 P 8050 2950
 F 0 "R7" V 7950 2900 50  0000 L CNN
-F 1 "330" V 8150 2900 50  0000 L CNN
+F 1 "1k" V 8150 2900 50  0000 L CNN
 F 2 "Resistor_THT:R_Axial_DIN0207_L6.3mm_D2.5mm_P10.16mm_Horizontal" H 8050 2950 50  0001 C CNN
 F 3 "~" H 8050 2950 50  0001 C CNN
@@
 Text Label 7500 2900 0    50   ~ 0
 DIGITAL4
-Text Label 2500 3800 0    50   ~ 0
+Text Label 1925 3525 0    50   ~ 0
 DIGITAL1
-Text Label 2500 3900 0    50   ~ 0
+Text Label 1925 3625 0    50   ~ 0
 DIGITAL2
 Wire Wire Line
 	3500 4950 3150 4950
-Text Label 2500 4000 0    50   ~ 0
+Text Label 1925 3725 0    50   ~ 0
 DIGITAL3
-Text Label 2500 4100 0    50   ~ 0
+Text Label 1925 3825 0    50   ~ 0
 DIGITAL4
 $Comp
 L power:GND #PWR01
 U 1 1 5DAD2345
-P 2550 4250
-F 0 "#PWR01" H 2550 4000 50  0001 C CNN
-F 1 "GND" H 2555 4077 50  0000 C CNN
-F 2 "" H 2550 4250 50  0001 C CNN
-F 3 "" H 2550 4250 50  0001 C CNN
-	1    2550 4250
-	1    0    0    -1
-$EndComp
-Wire Wire Line
-	2550 4250 2550 4200
-Wire Wire Line
-	2550 4200 2500 4200
+P 1975 3975
+F 0 "#PWR01" H 1975 3725 50  0001 C CNN
+F 1 "GND" H 1980 3802 50  0000 C CNN
+F 2 "" H 1975 3975 50  0001 C CNN
+F 3 "" H 1975 3975 50  0001 C CNN
+	1    1975 3975
+	1    0    0    -1
+$EndComp
+Wire Wire Line
+	1975 3975 1975 3925
+Wire Wire Line
+	1975 3925 1925 3925
 $Comp
 L power:GND #PWR02
 U 1 1 5DAD5216
-P 2900 3750
-F 0 "#PWR02" H 2900 3500 50  0001 C CNN
-F 1 "GND" H 2905 3577 50  0000 C CNN
-F 2 "" H 2900 3750 50  0001 C CNN
-F 3 "" H 2900 3750 50  0001 C CNN
-	1    2900 3750
-	1    0    0    -1
-$EndComp
-Wire Wire Line
-	2900 3750 2900 3700
-Wire Wire Line
-	2900 3700 2500 3700
+P 2325 3475
+F 0 "#PWR02" H 2325 3225 50  0001 C CNN
+F 1 "GND" H 2330 3302 50  0000 C CNN
+F 2 "" H 2325 3475 50  0001 C CNN
+F 3 "" H 2325 3475 50  0001 C CNN
+	1    2325 3475
+	1    0    0    -1
+$EndComp
+Wire Wire Line
+	2325 3475 2325 3425
+Wire Wire Line
+	2325 3425 1925 3425
 Wire Wire Line
 	3500 6900 3150 6900
@@
 L Connector_Generic:Conn_01x02 J6
 U 1 1 5DAE2C15
-P 2200 2650
-F 0 "J6" H 2120 2325 50  0000 C CNN
-F 1 "Conn_01x02" H 2120 2416 50  0000 C CNN
-F 2 "TerminalBlock:TerminalBlock_bornier-2_P5.08mm" H 2200 2650 50  0001 C CNN
-F 3 "~" H 2200 2650 50  0001 C CNN
-	1    2200 2650
+P 1725 2625
+F 0 "J6" H 1645 2300 50  0000 C CNN
+F 1 "Conn_01x02" H 1645 2391 50  0000 C CNN
+F 2 "TerminalBlock:TerminalBlock_bornier-2_P5.08mm" H 1725 2625 50  0001 C CNN
+F 3 "~" H 1725 2625 50  0001 C CNN
+	1    1725 2625
 	-1   0    0    1
 $EndComp
@@
 L power:+12V #PWR011
 U 1 1 5DAE2EF0
-P 2550 2450
-F 0 "#PWR011" H 2550 2300 50  0001 C CNN
-F 1 "+12V" H 2565 2623 50  0000 C CNN
-F 2 "" H 2550 2450 50  0001 C CNN
-F 3 "" H 2550 2450 50  0001 C CNN
-	1    2550 2450
-	1    0    0    -1
-$EndComp
-Wire Wire Line
-	2550 2450 2550 2500
-Wire Wire Line
-	2400 2550 2550 2550
+P 2075 2425
+F 0 "#PWR011" H 2075 2275 50  0001 C CNN
+F 1 "+12V" H 2090 2598 50  0000 C CNN
+F 2 "" H 2075 2425 50  0001 C CNN
+F 3 "" H 2075 2425 50  0001 C CNN
+	1    2075 2425
+	1    0    0    -1
+$EndComp
+Wire Wire Line
+	2075 2425 2075 2475
+Wire Wire Line
+	1925 2525 2075 2525
 $Comp
 L power:GND #PWR012
 U 1 1 5DAE636B
-P 2550 2750
-F 0 "#PWR012" H 2550 2500 50  0001 C CNN
-F 1 "GND" H 2555 2577 50  0000 C CNN
-F 2 "" H 2550 2750 50  0001 C CNN
-F 3 "" H 2550 2750 50  0001 C CNN
-	1    2550 2750
-	1    0    0    -1
-$EndComp
-Wire Wire Line
-	2550 2750 2550 2700
-Wire Wire Line
-	2550 2650 2400 2650
+P 2075 2725
+F 0 "#PWR012" H 2075 2475 50  0001 C CNN
+F 1 "GND" H 2080 2552 50  0000 C CNN
+F 2 "" H 2075 2725 50  0001 C CNN
+F 3 "" H 2075 2725 50  0001 C CNN
+	1    2075 2725
+	1    0    0    -1
+$EndComp
+Wire Wire Line
+	2075 2725 2075 2675
+Wire Wire Line
+	2075 2625 1925 2625
 $Comp
 L Device:C_Small C1
 U 1 1 5DAE5018
-P 2700 2600
-F 0 "C1" H 2792 2646 50  0000 L CNN
-F 1 "100n" H 2792 2555 50  0000 L CNN
-F 2 "Capacitor_THT:C_Disc_D5.0mm_W2.5mm_P5.00mm" H 2700 2600 50  0001 C CNN
-F 3 "~" H 2700 2600 50  0001 C CNN
-	1    2700 2600
-	1    0    0    -1
-$EndComp
-Wire Wire Line
-	2700 2500 2550 2500
-Connection ~ 2550 2500
-Wire Wire Line
-	2550 2500 2550 2550
-Wire Wire Line
-	2700 2700 2550 2700
-Connection ~ 2550 2700
-Wire Wire Line
-	2550 2700 2550 2650
+P 2225 2575
+F 0 "C1" H 2317 2621 50  0000 L CNN
+F 1 "100n" H 2317 2530 50  0000 L CNN
+F 2 "Capacitor_THT:C_Disc_D5.0mm_W2.5mm_P5.00mm" H 2225 2575 50  0001 C CNN
+F 3 "~" H 2225 2575 50  0001 C CNN
+	1    2225 2575
+	1    0    0    -1
+$EndComp
+Wire Wire Line
+	2225 2475 2075 2475
+Connection ~ 2075 2475
+Wire Wire Line
+	2075 2475 2075 2525
+Wire Wire Line
+	2225 2675 2075 2675
+Connection ~ 2075 2675
+Wire Wire Line
+	2075 2675 2075 2625
 $Comp
 L Device:CP_Small C2
 U 1 1 5DAEC27A
-P 3050 2600
-F 0 "C2" H 3138 2646 50  0000 L CNN
-F 1 "10uF" H 3138 2555 50  0000 L CNN
-F 2 "Capacitor_THT:CP_Radial_D8.0mm_P2.50mm" H 3050 2600 50  0001 C CNN
-F 3 "~" H 3050 2600 50  0001 C CNN
-	1    3050 2600
-	1    0    0    -1
-$EndComp
-Wire Wire Line
-	3050 2700 2700 2700
-Connection ~ 2700 2700
-Wire Wire Line
-	2700 2500 3050 2500
-Connection ~ 2700 2500
+P 2575 2575
+F 0 "C2" H 2663 2621 50  0000 L CNN
+F 1 "10uF" H 2663 2530 50  0000 L CNN
+F 2 "Capacitor_THT:CP_Radial_D8.0mm_P2.50mm" H 2575 2575 50  0001 C CNN
+F 3 "~" H 2575 2575 50  0001 C CNN
+	1    2575 2575
+	1    0    0    -1
+$EndComp
+Wire Wire Line
+	2575 2675 2225 2675
+Connection ~ 2225 2675
+Wire Wire Line
+	2225 2475 2575 2475
+Connection ~ 2225 2475
 $EndSCHEMATC
